Commit message: changed orientation of the gripper

File: urdf/camera_adapter.urdf.xacro (robot description, xacro)
@@ -7,5 +7,5 @@
         <parent link="${parent}" />
         <child link="camera_adapter_link" />
-        <origin xyz="0 0 0.005" rpy="0 0 ${J_PI}" />
+        <origin xyz="0 0 0.005" rpy="0 0 ${J_PI/2}" />
       </joint>
     </xacro:if>

Commit message: Added prefix

File: urdf/camera_adapter.urdf.xacro (robot description, xacro)
@@ -2,13 +2,13 @@
 <robot name="camera_adapter" xmlns:xacro="http://www.ros.org/wiki/xacro">
     <xacro:property name="J_PI" value="3.14159265359" />
-  <xacro:macro name="camera_adapter" params="parent:='' ">
+  <xacro:macro name="camera_adapter" params="parent:='' prefix:=''">
     <xacro:if value="${parent != ''}">
-      <joint name="camera_adapter_joint" type="fixed">
+      <joint name="${prefix}camera_adapter_joint" type="fixed">
         <parent link="${parent}" />
-        <child link="camera_adapter_link" />
+        <child link="${prefix}camera_adapter_link" />
         <origin xyz="0 0 0.005" rpy="0 0 ${J_PI/2}" />
       </joint>
     </xacro:if>
-    <link name="camera_adapter_link">
+    <link name="${prefix}camera_adapter_link">
       <inertial>
         <origin xyz="0 0 0.005" rpy="-${J_PI/2} 0 ${J_PI}" />
@@ -34,5 +34,5 @@
       </collision>
     </link>
-    <link name="camera_adapter_attach_link">
+    <link name="${prefix}camera_adapter_attach_link">
       <inertial>
         <origin xyz="0 0 0" rpy="0 0 0" />
@@ -43,7 +43,7 @@
       </inertial>
     </link>
-    <joint name="camera_adapter_attach_joint" type="fixed">
-      <parent link="camera_adapter_link" />
-      <child link="camera_adapter_attach_link" />
+    <joint name="${prefix}camera_adapter_attach_joint" type="fixed">
+      <parent link="${prefix}camera_adapter_link" />
+      <child link="${prefix}camera_adapter_attach_link" />
       <origin xyz="0 0 0.005" rpy="0 0 0"  />
     </joint>

File: urdf/gripper.urdf.xacro (robot description, xacro)
@@ -1,14 +1,14 @@
 <?xml version="1.0" encoding='utf-8'?>
 <robot name="zimmer_gripper" xmlns:xacro="http://www.ros.org/wiki/xacro">
-  <xacro:macro name="zimmer_gripper" params="parent:='' ">
+  <xacro:macro name="zimmer_gripper" params="parent:='' prefix:=''">
     <xacro:include
       filename="$(find zimmer_gripper_description)/urdf/zimmer_gripper.transmission.xacro" />
     <xacro:include filename="$(find zimmer_gripper_description)/urdf/zimmer_gripper.gazebo.xacro" />
-    <joint name="gripper_joint" type="fixed">
+    <joint name="${prefix}gripper_joint" type="fixed">
       <parent link="${parent}" />
-      <child link="zimmer_gripper_body" />
+      <child link="${prefix}zimmer_gripper_body" />
       <origin xyz="0 -0.039 0" rpy="0 1.5708 0" />
     </joint>
-    <link name="zimmer_gripper_body">
+    <link name="${prefix}zimmer_gripper_body">
       <inertial>
         <origin xyz="0 -0.039 0" rpy="0 1.5708 0" />
@@ -32,5 +32,5 @@
       </collision>
     </link>
-    <link name="zimmer_gripper_left_finger">
+    <link name="${prefix}zimmer_gripper_left_finger">
       <inertial>
         <origin rpy="0 0 0" xyz="0 0.01 0.02" />
@@ -56,5 +56,5 @@
       </collision>
     </link>
-    <link name="zimmer_gripper_right_finger">
+    <link name="${prefix}zimmer_gripper_right_finger">
       <inertial>
         <origin rpy="0 0 0" xyz="0 0.01 0.02" />
@@ -98,26 +98,26 @@
       <implicitSpringDamper>True</implicitSpringDamper>
     </joint> -->
-    <joint name="zimmer_finger_left" type="fixed">
-      <parent link="zimmer_gripper_body" />
-      <child link="zimmer_gripper_left_finger" />
+    <joint name="${prefix}zimmer_finger_left" type="fixed">
+      <parent link="${prefix}zimmer_gripper_body" />
+      <child link="${prefix}zimmer_gripper_left_finger" />
       <origin rpy="0 0 0" xyz="0 0 0" />
     </joint>
-    <joint name="zimmer_finger_right" type="fixed">
-      <parent link="zimmer_gripper_body" />
-      <child link="zimmer_gripper_right_finger" />
+    <joint name="${prefix}zimmer_finger_right" type="fixed">
+      <parent link="${prefix}zimmer_gripper_body" />
+      <child link="${prefix}zimmer_gripper_right_finger" />
       <origin rpy="0 0 0" xyz="0 0 0" />
     </joint>
-    <xacro:mimic_joint_plugin_gazebo name_prefix="zimmer_finger_right"
-      parent_joint="zimmer_finger_left"
-      mimic_joint="zimmer_finger_right"
+    <xacro:mimic_joint_plugin_gazebo name_prefix="${prefix}zimmer_finger_right"
+      parent_joint="${prefix}zimmer_finger_left"
+      mimic_joint="${prefix}zimmer_finger_right"
       has_pid="false"
       multiplier="1.0"
       max_effort="2000" />
-    <joint name="connection_joint" type="fixed">
+    <joint name="§(prefix)connection_joint" type="fixed">
       <origin xyz="0 -0.128 0" rpy="0 0 0" />
-      <parent link="zimmer_gripper_body" />
-      <child link="zimmer_gripper_tcp" />
+      <parent link="${prefix}zimmer_gripper_body" />
+      <child link="${prefix}zimmer_gripper_tcp" />
     </joint>
-    <link name="zimmer_gripper_tcp" />
+    <link name="${prefix}zimmer_gripper_tcp" />
   </xacro:macro>
 </robot>

Commit message: added the camera

File: urdf/camera_adapter.urdf.xacro (robot description, xacro)
@@ -48,4 +48,18 @@
       <origin xyz="0 0 0.005" rpy="0 0 0"  />
     </joint>
+    <link name="${prefix}camera_adapter_mount_link">
+      <inertial>
+        <origin xyz="0 0 0" rpy="0 0 0" />
+        <mass value="0.00" />
+        <inertia ixx="0.0" ixy="0.0" ixz="0.0"
+          iyy="0.0" iyz="0.0"
+          izz="0.0" />
+      </inertial>
+    </link>
+    <joint name="${prefix}camera_adapter_mount_joint" type="fixed">
+      <parent link="${prefix}camera_adapter_attach_link" />
+      <child link="${prefix}camera_adapter_mount_link" />
+      <origin xyz="0 0.08 0" rpy="0 0 0" />
+    </joint>
   </xacro:macro>
 </robot>

File: urdf/zimmer_gripper.urdf.xacro (robot description, xacro)
@@ -2,14 +2,20 @@
 <robot name="zimmer_gripper" xmlns:xacro="http://www.ros.org/wiki/xacro" >
   <xacro:property name="J_PI" value="3.14159265359" />
+  <xacro:include filename="$(find zimmer_gripper_description)/urdf/camera_adapter.urdf.xacro"/>
   <xacro:include filename="$(find zimmer_gripper_description)/urdf/match.urdf.xacro"/>
   <xacro:include filename="$(find zimmer_gripper_description)/urdf/gripper.urdf.xacro"/>
+  <xacro:include filename="$(find intel_realsense_d435i_description)/urdf/d435i.urdf.xacro"/>
   <link name="world" />
   <joint name="world_joint" type="fixed">
     <origin xyz="0 0 0" rpy="-${J_PI/2} 0 0"/>
     <parent link="world" />
-    <child link="zimmer_match_link" />
+    <child link="camera_adapter_link" />
   </joint>
-  <xacro:zimmer_match parent=''/>
+  <xacro:camera_adapter parent='' />
+  <xacro:zimmer_match parent='camera_adapter_attach_link'/>
   <xacro:zimmer_gripper parent='zimmer_match_link' />
+    <xacro:sensor_d435 name="camera" topics_ns="camera" parent="camera_adapter_mount_link" publish_pointcloud="true">
+    <origin xyz="0 -0.0125 0.01" rpy="${J_PI/2} -${J_PI/2} ${J_PI}" />
+  </xacro:sensor_d435>
   <gazebo>
     <plugin name="gazebo_ros_control" filename="libgazebo_ros_control.so">

Commit message: Added minium mass and inertias for Gazebo

File: urdf/camera_adapter.urdf.xacro (robot description, xacro)
@@ -1,5 +1,5 @@
 <?xml version="1.0" encoding="utf-8"?>
 <robot name="camera_adapter" xmlns:xacro="http://www.ros.org/wiki/xacro">
-    <xacro:property name="J_PI" value="3.14159265359" />
+  <xacro:property name="J_PI" value="3.14159265359" />
   <xacro:macro name="camera_adapter" params="parent:='' prefix:=''">
     <xacro:if value="${parent != ''}">
@@ -13,8 +13,8 @@
       <inertial>
         <origin xyz="0 0 0.005" rpy="-${J_PI/2} 0 ${J_PI}" />
-        <mass value="0.00" />
-        <inertia ixx="0.0" ixy="0.0" ixz="0.0"
-          iyy="0.0" iyz="0.0"
-          izz="0.0" />
+        <mass value="0.1" />
+        <inertia ixx="0.0001" ixy="0.0" ixz="0.0"
+          iyy="0.0001" iyz="0.0"
+          izz="0.0001" />
       </inertial>
       <visual>
@@ -37,8 +37,8 @@
       <inertial>
         <origin xyz="0 0 0" rpy="0 0 0" />
-        <mass value="0.00" />
-        <inertia ixx="0.0" ixy="0.0" ixz="0.0"
-          iyy="0.0" iyz="0.0"
-          izz="0.0" />
+        <mass value="0.01" />
+        <inertia ixx="0.000001" ixy="0.0" ixz="0.0"
+          iyy="0.000001" iyz="0.0"
+          izz="0.000001" />
       </inertial>
     </link>
@@ -51,8 +51,8 @@
       <inertial>
         <origin xyz="0 0 0" rpy="0 0 0" />
-        <mass value="0.00" />
-        <inertia ixx="0.0" ixy="0.0" ixz="0.0"
-          iyy="0.0" iyz="0.0"
-          izz="0.0" />
+        <mass value="0.01" />
+        <inertia ixx="0.000001" ixy="0.0" ixz="0.0"
+          iyy="0.000001" iyz="0.0"
+          izz="0.000001" />
       </inertial>
     </link>
