Commit message: changed to fixed joints

File: urdf/gripper.urdf.xacro (robot description, xacro)
@@ -80,5 +80,5 @@
       </collision>
     </link>
-    <joint name="zimmer_finger_left" type="prismatic">
+    <!-- <joint name="zimmer_finger_left" type="prismatic">
       <parent link="zimmer_gripper_body" />
       <child link="zimmer_gripper_left_finger" />
@@ -97,4 +97,14 @@
       <dynamics damping="0.1" friction="0.0" />
       <implicitSpringDamper>True</implicitSpringDamper>
+    </joint> -->
+    <joint name="zimmer_finger_left" type="fixed">
+      <parent link="zimmer_gripper_body" />
+      <child link="zimmer_gripper_left_finger" />
+      <origin rpy="0 0 0" xyz="0 0 0" />
+    </joint>
+    <joint name="zimmer_finger_right" type="fixed">
+      <parent link="zimmer_gripper_body" />
+      <child link="zimmer_gripper_right_finger" />
+      <origin rpy="0 0 0" xyz="0 0 0" />
     </joint>
     <xacro:mimic_joint_plugin_gazebo name_prefix="zimmer_finger_right"

Commit message: edit the weight of the gripper

File: urdf/gripper.urdf.xacro (robot description, xacro)
@@ -13,5 +13,5 @@
       <inertial>
         <origin xyz="0 -0.039 0" rpy="0 1.5708 0" />
-        <mass value="0.76" />
+        <mass value="0.576" />
         <inertia ixx="0.0" ixy="0.0" ixz="0.0" iyy="0.0" iyz="0.0" izz="0.0" />
       </inertial>

Commit message: Changed gripper weight

File: urdf/gripper.urdf.xacro (robot description, xacro)
@@ -13,5 +13,5 @@
       <inertial>
         <origin xyz="0 -0.039 0" rpy="0 1.5708 0" />
-        <mass value="0.576" />
+        <mass value="0.76" />
         <inertia ixx="0.0" ixy="0.0" ixz="0.0" iyy="0.0" iyz="0.0" izz="0.0" />
       </inertial>

Commit message: MAde the zimmer_gripper an macro

File: urdf/gripper.urdf.xacro (robot description, xacro)
@@ -80,7 +80,7 @@
       </collision>
     </link>
-    <!-- <joint name="zimmer_finger_left" type="prismatic">
-      <parent link="zimmer_gripper_body" />
-      <child link="zimmer_gripper_left_finger" />
+    <joint name="${prefix}zimmer_finger_left" type="prismatic">
+      <parent link="${prefix}zimmer_gripper_body" />
+      <child link="${prefix}zimmer_gripper_left_finger" />
       <origin rpy="0 0 0" xyz="0 0 0" />
       <axis xyz="0 0 -1" />
@@ -88,23 +88,13 @@
     </joint>
     <xacro:insert_transmission name="zimmer_finger_left" />
-    <joint name="zimmer_finger_right" type="prismatic">
-      <parent link="zimmer_gripper_body" />
-      <child link="zimmer_gripper_right_finger" />
+    <joint name="${prefix}zimmer_finger_right" type="prismatic">
+      <parent link="${prefix}zimmer_gripper_body" />
+      <child link="${prefix}zimmer_gripper_right_finger" />
       <origin rpy="0 0 0" xyz="0 0 0" />
       <axis xyz="0 0 1" />
-      <mimic joint="zimmer_finger_left" multiplier="1" />
+      <mimic joint="${prefix}zimmer_finger_left" multiplier="1" />
       <limit effort="2000" lower="0" upper="0.016" velocity="0.2" />
       <dynamics damping="0.1" friction="0.0" />
       <implicitSpringDamper>True</implicitSpringDamper>
-    </joint> -->
-    <joint name="${prefix}zimmer_finger_left" type="fixed">
-      <parent link="${prefix}zimmer_gripper_body" />
-      <child link="${prefix}zimmer_gripper_left_finger" />
-      <origin rpy="0 0 0" xyz="0 0 0" />
-    </joint>
-    <joint name="${prefix}zimmer_finger_right" type="fixed">
-      <parent link="${prefix}zimmer_gripper_body" />
-      <child link="${prefix}zimmer_gripper_right_finger" />
-      <origin rpy="0 0 0" xyz="0 0 0" />
     </joint>
     <xacro:mimic_joint_plugin_gazebo name_prefix="${prefix}zimmer_finger_right"

File: urdf/zimmer_gripper.urdf.xacro (robot description, xacro)
@@ -1,25 +1,14 @@
 <?xml version="1.0" encoding='utf-8'?>
 <robot name="zimmer_gripper" xmlns:xacro="http://www.ros.org/wiki/xacro" >
-  <xacro:property name="J_PI" value="3.14159265359" />
-  <xacro:include filename="$(find zimmer_gripper_description)/urdf/camera_adapter.urdf.xacro"/>
   <xacro:include filename="$(find zimmer_gripper_description)/urdf/match.urdf.xacro"/>
   <xacro:include filename="$(find zimmer_gripper_description)/urdf/gripper.urdf.xacro"/>
-  <xacro:include filename="$(find camera_description)/urdf/d435i.urdf.xacro"/>
-  <link name="world" />
-  <joint name="world_joint" type="fixed">
-    <origin xyz="0 0 0" rpy="-${J_PI/2} 0 0"/>
-    <parent link="world" />
-    <child link="camera_adapter_link" />
-  </joint>
-  <xacro:camera_adapter parent='' />
-  <xacro:zimmer_match parent='camera_adapter_attach_link'/>
-  <xacro:zimmer_gripper parent='zimmer_match_link' />
-    <xacro:sensor_d435 name="camera" topics_ns="camera" parent="camera_adapter_mount_link" publish_pointcloud="true">
-    <origin xyz="0 -0.0125 0.01" rpy="${J_PI/2} -${J_PI/2} ${J_PI}" />
-  </xacro:sensor_d435>
-  <gazebo>
-    <plugin name="gazebo_ros_control" filename="libgazebo_ros_control.so">
-      <robotNamespace>/</robotNamespace>
-    </plugin>
-  </gazebo>
+  <xacro:macro name="zimmer_gripper_macro" params="parent">
+    <xacro:zimmer_match parent='${parent}'/>
+    <xacro:zimmer_gripper parent='zimmer_match_link' />
+    <gazebo>
+      <plugin name="gazebo_ros_control" filename="libgazebo_ros_control.so">
+        <robotNamespace>/</robotNamespace>
+      </plugin>
+    </gazebo>
+  </xacro:macro>
 </robot>

Commit message: Modify the movement of the gripper fingers.

File: urdf/gripper.urdf.xacro (robot description, xacro)
@@ -84,15 +84,15 @@
       <child link="${prefix}zimmer_gripper_left_finger" />
       <origin rpy="0 0 0" xyz="0 0 0" />
-      <axis xyz="0 0 -1" />
-      <limit effort="2000" lower="0.0" upper="0.016" velocity="0.2" />
+      <axis xyz="0 0 1" />
+      <limit effort="2000" lower="-0.016" upper="0.0" velocity="0.2" />
     </joint>
-    <xacro:insert_transmission name="zimmer_finger_left" />
+      <xacro:insert_transmission name="zimmer_finger_left" />
     <joint name="${prefix}zimmer_finger_right" type="prismatic">
       <parent link="${prefix}zimmer_gripper_body" />
       <child link="${prefix}zimmer_gripper_right_finger" />
       <origin rpy="0 0 0" xyz="0 0 0" />
-      <axis xyz="0 0 1" />
+      <axis xyz="0 0 -1" />
       <mimic joint="${prefix}zimmer_finger_left" multiplier="1" />
-      <limit effort="2000" lower="0" upper="0.016" velocity="0.2" />
+      <limit effort="2000" lower="-0.016" upper="0.0" velocity="0.2" />
       <dynamics damping="0.1" friction="0.0" />
       <implicitSpringDamper>True</implicitSpringDamper>
